File: pcb/speaker.kicad_sch (KiCad schematic)
At the start: 2 parts, among them J10 AudioJack2

Commit message: update vca
Parts:
- J10: footprint (none) -> Connector_Audio:Jack_3.5mm_CUI_SJ1-3513N_Horizontal
- RV7: footprint (none) -> Potentiometer_THT:Potentiometer_Bourns_PTV09A-1_Single_Vertical
Changed lines of the file:
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@@
 			)
 		)
-		(property "Footprint" ""
+		(property "Footprint" "Connector_Audio:Jack_3.5mm_CUI_SJ1-3513N_Horizontal"
 			(at 166.37 100.33 0)
 			(effects
@@
 			)
 		)
-		(property "Footprint" ""
+		(property "Footprint" "Potentiometer_THT:Potentiometer_Bourns_PTV09A-1_Single_Vertical"
 			(at 147.32 100.33 0)
 			(effects
