File: pcb/one-voice-synth.kicad_sch (KiCad schematic)
At the start: 12 parts, among them J1 Conn_01x02, J11 Conn_01x04, J2 Conn_01x02, J3 Conn_01x02, J4 Conn_01x02, J6 Conn_01x02, J7 Conn_01x02, J8 Conn_01x03, P1 USB_C_Plug_USB2.0, U6 TL072

Commit message: update vca
Parts:
- removed P1: USB_C_Plug_USB2.0, symbol Connector:USB_C_Plug_USB2.0
- removed R34, R35: 100k, symbol Device:R
- removed U6: TL072, symbol Amplifier_Operational:TL072
- J1, J2, J3, J4, J6, J7: footprint (none) -> Connector_PinHeader_2.54mm:PinHeader_1x02_P2.54mm_Vertical
- J11: footprint (none) -> Connector_PinHeader_2.54mm:PinHeader_1x04_P2.54mm_Vertical
- J8: footprint (none) -> Connector_PinHeader_2.54mm:PinHeader_1x03_P2.54mm_Horizontal
Other:
- sheet Low-Pass Filter renamed a
- note removed: "Split-rail ground"
- note removed: "UNUSED"
- note removed: "Use 1% resistors"

Commit message: Update rails, start to clean
Parts:
- J11, J8: now not fitted
Connections:
- net +2V5 is gone; now on net +9V: J11.2 (Pin_2)
- net -2V5 is gone; now on net -9V: J11.1 (Pin_1)
Other:
- sheet a renamed Low-pass Filter
